File: hatecbse.kicad_sch (KiCad schematic)
At the start: 18 parts, among them J1 Screw_Terminal_01x06, J2 Screw_Terminal_01x06, J3 Barrel_Jack_MountingPin, J4 Conn_01x04_Socket, J5 Conn_01x03, J6 Conn_01x02_Pin, J7 Conn_01x02_Pin, J8 Conn_01x04_Pin, U1 TMC2209_SILENTSTEPSTICK, U2 TMC2209_SILENTSTEPSTICK

Commit message: diddy
Parts:
- removed A1: RaspberryPi_Pico, Module:RaspberryPi_Pico_Common_Unspecified, symbol MCU_Module:RaspberryPi_Pico
- removed D1, D2: LED, LED_THT:LED_D3.0mm, symbol Device:LED
- removed R1: 1.2k, Resistor_THT:R_Axial_DIN0204_L3.6mm_D1.6mm_P1.90mm_Vertical, symbol Device:R
- removed R2: 500, Resistor_THT:R_Axial_DIN0204_L3.6mm_D1.6mm_P1.90mm_Vertical, symbol Device:R
- added C1, C21, C24, C25, C26, C27, C28, C29, C30, C31, C32, C33, C6: 100 n, Capacitor_SMD:C_0402_1005Metric, symbol Device:C
- added C16, C20: 10 u, Capacitor_SMD:C_0402_1005Metric, symbol Device:C
- added C17, C18, C19, C5: 4.7 u, Capacitor_SMD:C_0402_1005Metric, symbol Device:C
- added C22, C23: 15 p, Capacitor_SMD:C_0402_1005Metric, symbol Device:C
- added C7: 10 uF, Capacitor_SMD:C_0402_1005Metric, symbol Device:C
- added D3, D4, D5: LED, LED_THT:LED_D3.0mm, symbol Device:LED
- added H1, H2, H3, H4: MountingHole, MountingHole:MountingHole_3.2mm_M3, symbol Mechanical:MountingHole
- added J10: Conn_01x20_Pin, Connector_PinSocket_2.54mm:PinSocket_1x20_P2.54mm_Vertical, symbol Connector:Conn_01x20_Pin
- added J12, J13, J14, J15, J16, J17: Conn_01x02_Pin, Connector_PinSocket_2.54mm:PinSocket_1x02_P2.54mm_Vertical, symbol Connector:Conn_01x02_Pin
- added J9: USB_C_Receptacle_USB2.0_14P, Connector_USB:USB_C_Receptacle_XKB_U262-16XN-4BVC11, symbol Connector:USB_C_Receptacle_USB2.0_14P
- added L1: 3.3 u, Inductor_SMD:L_0805_2012Metric, symbol Device:L
- added R10: 0, Resistor_SMD:R_0805_2012Metric, symbol Device:R
- added R11, R12: DNF, symbol Device:R
- added R13, R3, R5: 1k, Resistor_SMD:R_0402_1005Metric, symbol Device:R
- added R14: 1.2k, Resistor_THT:R_Axial_DIN0204_L3.6mm_D1.6mm_P1.90mm_Vertical, symbol Device:R
- added R15: 500, Resistor_THT:R_Axial_DIN0204_L3.6mm_D1.6mm_P1.90mm_Vertical, symbol Device:R
- added R16: 330, Resistor_THT:R_Axial_DIN0204_L3.6mm_D1.6mm_P1.90mm_Vertical, symbol Device:R
- added R17, R18: 33R, Resistor_SMD:R_0402_1005Metric, symbol Device:R
- added R19, R20: 27, Resistor_SMD:R_0201_0603Metric, symbol Device:R
- added R4: 33, Resistor_SMD:R_0201_0603Metric, symbol Device:R
- added R8, R9: 5.1k, Resistor_SMD:R_0603_1608Metric, symbol Device:R
- added SW1, SW2: SW_Push, Button_Switch_SMD:SW_Tactile_SPST_NO_Straight_CK_PTS636Sx25SMTRLFS, symbol Switch:SW_Push
- added U3: RP2350B, Package_DFN_QFN:QFN-80-1EP_10x10mm_P0.4mm_EP3.4x3.4mm, symbol MCU_RaspberryPi:RP2350B
- added U4: NCP1117-3.3_SOT223, Package_TO_SOT_SMD:SOT-223-3_TabPin2, symbol Regulator_Linear:NCP1117-3.3_SOT223
- added U5: W25Q128JVS, Package_SO:SOIC-8_5.3x5.3mm_P1.27mm, symbol Memory_Flash:W25Q128JVS
- added U6: USBLC6-2SC6, Package_TO_SOT_SMD:SOT-23-6, symbol Power_Protection:USBLC6-2SC6
- added Y1: Crystal_GND24, Crystal:Crystal_SMD_Abracon_ABM8G-4Pin_3.2x2.5mm, symbol Device:Crystal_GND24
Connections:
- net +12V: now also J2.1 (Pin_1), J14.1 (Pin_1), J15.1 (Pin_1), R14.1; no longer J2.6 (Pin_6)
- net +5V: now also C16.1, J16.1 (Pin_1), J17.1 (Pin_1), J9.A4 (VBUS), J9.A9 (VBUS), J9.B4 (VBUS), J9.B9 (VBUS), R15.1, U4.3 (VI), U6.5 (VBUS)
- net DIR_1: now also J10.12 (Pin_12), U3.9 (GPIO11)
- net DIR_2: now also J10.14 (Pin_14), U3.12 (GPIO13)
- net EN_1: now also J10.10 (Pin_10), U3.7 (GPIO9)
- net EN_2: now also J10.9 (Pin_9), U3.6 (GPIO8)
- net GND: now also J2.6 (Pin_6), C1.2, C16.2, C17.1, C18.2, C19.2, C20.2, C21.2, C22.1, C23.1, C24.2, C25.2, C26.2, C27.2, C28.2, C29.2, C30.2, C31.2, C32.2, C33.2, C5.2, C6.2, C7.2, D3.2 (A), D4.2 (A), D5.2 (A), J10.4 (Pin_4), J12.2 (Pin_2), J13.2 (Pin_2), J14.2 (Pin_2), J15.2 (Pin_2), J16.2 (Pin_2), J17.2 (Pin_2), J9.A1 (GND), J9.A12 (GND), J9.B1 (GND), J9.B12 (GND), J9.SH (SHIELD), R3.2, R8.2, R9.2, SW2.1, U3.62 (VREG_PGND), U3.81 (GND), U4.1 (GND), U5.4 (GND), U6.2 (GND), Y1.2 (G), Y1.4 (G); no longer J2.1 (Pin_1)
- net LS_1: now also J10.6 (Pin_6), U3.2 (GPIO5)
- net LS_2: now also J10.7 (Pin_7), U3.3 (GPIO6)
- net M2_1A: now also J2.5 (Pin_5); no longer J2.2 (Pin_2)
- net M2_1B: now also J2.3 (Pin_3); no longer J2.4 (Pin_4)
- net M2_2A: now also J2.4 (Pin_4); no longer J2.3 (Pin_3)
- net M2_2B: now also J2.2 (Pin_2); no longer J2.5 (Pin_5)
- net SCL: now also J10.1 (Pin_1), U3.77 (GPIO0)
- net SDA: now also J10.2 (Pin_2), U3.78 (GPIO1)
- net SERVO: now also J10.8 (Pin_8), U3.4 (GPIO7)
- net STEP_1: now also J10.11 (Pin_11), U3.8 (GPIO10)
- net STEP_2: now also J10.13 (Pin_13), U3.11 (GPIO12)
- new net: J9.A5 (CC1), R8.1
- new net: J9.A6 (D+), J9.B6 (D+), U6.3 (I/O2)
- new net: J9.A7 (D-), J9.B7 (D-), U6.1 (I/O1)
- new net: J9.B5 (CC2), R9.1
- new net: R5.2, SW2.2
- new net: R18.1, U6.4 (I/O2)
- new net: R17.1, U6.6 (I/O1)
- new net: D4.1 (K), R15.2
- new net: C22.2, R13.1, Y1.3
- new net: R10.2, R11.2, R12.2, U5.1 (~{CS})
- new net: D3.1 (K), R14.2
- new net: D5.1 (K), R16.2
- new net: R3.1, SW1.1
- new net: R18.2, R20.2
- new net: SW1.2, U3.35 (RUN)
- new net: R17.2, R19.2
- new net +1V1: C1.1, C18.1, C5.1, C6.1, L1.1, U3.10 (DVDD), U3.32 (DVDD), U3.51 (DVDD), U3.65 (VREG_FB)
- new net +3V3: C19.1, C20.1, C21.1, C24.1, C25.1, C26.1, C27.1, C28.1, C29.1, C30.1, C31.1, C32.1, C33.1, C7.1, J10.3 (Pin_3), J12.1 (Pin_1), J13.1 (Pin_1), R12.1, R16.1, R4.2, U3.15 (IOVDD), U3.24 (IOVDD), U3.29 (IOVDD), U3.41 (IOVDD), U3.5 (IOVDD), U3.50 (IOVDD), U3.59 (ADC_AVDD), U3.60 (IOVDD), U3.64 (VREG_VIN), U3.68 (USB_OTP_VDD), U3.69 (QSPI_IOVDD), U3.76 (IOVDD), U4.2 (VO), U5.8 (VCC)
- new net GPIO0: R11.1
- new net GPIO14: J10.15 (Pin_15), U3.13 (GPIO14)
- new net GPIO15: J10.16 (Pin_16), U3.14 (GPIO15)
- new net GPIO16: J10.17 (Pin_17), U3.16 (GPIO16)
- new net GPIO17: J10.18 (Pin_18), U3.17 (GPIO17)
- new net GPIO18: J10.19 (Pin_19), U3.18 (GPIO18)
- new net GPIO19: J10.20 (Pin_20), U3.19 (GPIO19)
- new net GPIO2: U3.79 (GPIO2)
- new net GPIO3: U3.80 (GPIO3)
- new net GPIO4: J10.5 (Pin_5), U3.1 (GPIO4)
- new net QSPI_SCLK: U3.71 (QSPI_SCLK), U5.6 (CLK)
- new net QSPI_SD1: U3.74 (QSPI_SD1), U5.2 (DO/IO_{1})
- new net QSPI_SD2: U3.73 (QSPI_SD2), U5.3 (~{WP}/IO_{2})
- new net QSPI_SD3: U3.70 (QSPI_SD3), U5.7 (~{HOLD}/~{RESET}/IO_{3})
- new net QSPI_SDO: U3.72 (QSPI_SD0), U5.5 (DI/IO_{0})
- new net USB_BOOT: R5.1, U3.75 (~{QSPI_SS})
- new net USB_D+: R20.1, U3.67 (USB_DP)
- new net USB_D-: R19.1, U3.66 (USB_DM)
- new net VREG_AVDD: C17.2, R4.1, U3.61 (VREG_AVDD)
- new net VREG_LX: L1.2, U3.63 (VREG_LX)
- new net XIN: C23.2, U3.30 (XIN), Y1.1
- new net XOUT: R13.2, U3.31 (XOUT)
- no-connect marks 27 -> 32
Other:
- note added: "MCU + FLASH"
- note added: "USB + VBUS"
- note removed: "MCU"
- moved on the sheet: C2, C3, C4, J1, J2, J3, J4, J5, J6, J7, J8, U1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
